File: machxo2_design_kicad/FPGA Power & Decoupling.kicad_sch (KiCad schematic)
At the start: 10 parts, among them U3 LCMX02-256HC-4SG32C

Commit message: Schematic bom generated. Preliminary review down. Layout started.
Parts:
- C14, C15, C17, C18, C19, C20, C21, C22: footprint (none) -> Capacitor_SMD:C_0402_1005Metric; Link (none) -> https://www.digikey.com/en/products/detail/murata-electroni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; Part Number (none) -> GRM155R61A104KA01J
- C16: footprint (none) -> Capacitor_SMD:C_0402_1005Metric; Link (none) -> https://www.digikey.com/en/products/detail/murata-electroni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; Part Number (none) -> GRM155R61A106ME11D
- U3: Link https://www.digikey.com/en/products/detail/lattice-semiconductor-corporation/LCMXO2-256HC-4SG32C/3232671?s=N4IgTCBcDaIDYGMC2APA9mAtGArANgAsFMAWAZwHMBmMBEAXQF8g -> https://www.digikey.com/en/products/detail/lattice-semiconductor-corporation/lcmxo2-256hc-4sg32c/3232671; Part Number (none) -> LCMXO2-256HC-4SG32C
